File: sensorweb-nodeMCU/sensorweb-nodeMCU.kicad_pcb (KiCad board)
At the start: 2 copper layers, 50.8 x 53.3 mm, 19 parts, among them P1 PMS3003, Q1 2N2222, U1 LT1302CN8-5

Commit message: Fixing schematic and PCB
Parts:
- removed B1: +VBAT, Wire_Pads:SolderWirePad_single_0-8mmDrill
- removed B2: -VBAT, Wire_Pads:SolderWirePad_single_0-8mmDrill
- added +VBAT: +VBAT, Wire_Pads:SolderWirePad_single_0-8mmDrill, F.Cu at (86.4, 101.6)
- added -VBAT: -VBAT, Wire_Pads:SolderWirePad_single_0-8mmDrill, F.Cu at (86.4, 104.1)
- added ?: PCB_mount, Wire_Pads:SolderWirePad_single_2-5mmDrill, F.Cu at (124.5, 82.5)
- added ?: PCB_mount, Wire_Pads:SolderWirePad_single_2-5mmDrill, F.Cu at (78.7, 82.5)
- added ?: PCB_mount, Wire_Pads:SolderWirePad_single_2-5mmDrill, F.Cu at (124.5, 130.8)
- added ?: PCB_mount, Wire_Pads:SolderWirePad_single_2-5mmDrill, F.Cu at (78.7, 130.8)
- added REF**: BatAtt., Wire_Pads:SolderWirePad_single_1-5mmDrill, F.Cu at (80.0, 104.1)
- added REF**: BatAtt., Wire_Pads:SolderWirePad_single_1-5mmDrill, F.Cu at (80.0, 101.6)
- L1: footprint Inductors:INDUCTOR_V -> Inductors_NEOSID:Neosid_Inductor_Sd14
- Q1: footprint TO_SOT_Packages_THT:TO-18_3Pin -> TO_SOT_Packages_THT:TO-92_Inline_Narrow_Oval
- moved Q1 23.9 mm to (101.6, 124.5), turned to 90 degrees
- moved C1 22.6 mm to (106.7, 90.2)
- moved L1 19.9 mm to (115.6, 88.9), turned to 90 degrees
- moved C8 19.4 mm to (101.6, 114.3), turned to 270 degrees
- moved C5 19.2 mm to (96.5, 96.5), turned to 270 degrees
- moved C7 18.0 mm to (106.7, 102.9), turned to 180 degrees
- moved R3 17.3 mm to (119.4, 99.1)
- moved C2 15.2 mm to (106.7, 85.1), turned to 180 degrees
- moved R2 10.9 mm to (90.2, 114.3), turned to 270 degrees
- moved R1 7.73 mm to (95.2, 114.3), turned to 270 degrees
- moved C3 5.24 mm to (106.7, 95.2), turned to 180 degrees
- moved D1 4.02 mm to (110.5, 102.9), turned to 0 degrees
- moved C4 2.54 mm to (86.4, 83.8)
- moved C6 1.80 mm to (86.4, 92.7)
- moved U1 1.80 mm to (95.2, 86.4)
Connections:
- C3 pad 1: Net-(C3-Pad1) -> +5V
- C5 pad 1: GND -> Net-(B1-Pad1)
- C5 pad 2: Net-(B1-Pad1) -> GND
- D1 pad 2: Net-(C3-Pad1) -> Net-(D1-Pad2)
- L1 pad 1: Net-(C3-Pad1) -> Net-(D1-Pad2)
- P1 pad 1: +5V -> (no net)
- P1 pad 2: GND -> (no net)
- P1 pad 3: Net-(P1-Pad3) -> (no net)
- P1 pad 4: Net-(MCU1-Pad18) -> Net-(MCU1-Pad19)
- P1 pad 5: Net-(MCU1-Pad19) -> Net-(MCU1-Pad18)
- P1 pad 6: (no net) -> Net-(P1-Pad6)
- P1 pad 7: (no net) -> GND
- P1 pad 8: (no net) -> +5V
- Q1 pad 1: Net-(Q1-Pad1) -> GND
- Q1 pad 2: Net-(P1-Pad3) -> Net-(Q1-Pad2)
- Q1 pad 3: GND -> Net-(P1-Pad6)
- R1 pad 1: Net-(Q1-Pad1) -> Net-(Q1-Pad2)
- R2 pad 2: Net-(P1-Pad3) -> Net-(P1-Pad6)
- U1 pad 7: Net-(C3-Pad1) -> Net-(D1-Pad2)
Routing:
- net Net-(P1-Pad6): track 0.00 -> 50.8 mm
- net Net-(P1-Pad3): track 35.6 -> 0.00 mm
- net Net-(D1-Pad2): track 0.00 -> 35.4 mm, vias 0 -> 1
- net Net-(C3-Pad1): track 21.7 -> 0.00 mm
- net Net-(Q1-Pad1): track 16.1 -> 0.00 mm
- net Net-(B1-Pad1): track 71.2 -> 56.5 mm
- net Net-(Q1-Pad2): track 0.00 -> 14.1 mm
- net GND: track 115.7 -> 129.3 mm, vias 0 -> 1
- net Net-(MCU1-Pad18): track 55.3 -> 64.1 mm
- net Net-(C7-Pad1): track 31.1 -> 39.5 mm, vias 0 -> 1
- net Net-(MCU1-Pad13): track 40.1 -> 46.7 mm
- net Net-(MCU1-Pad27): track 16.0 -> 19.4 mm
- net +5V: track 95.1 -> 95.8 mm
- net Net-(C4-Pad1): track 11.7 -> 12.5 mm
- net Net-(MCU1-Pad19): track 52.6 -> 52.0 mm, vias 2 -> 0
Other:
- board text added: "USB"
