File: sensorweb-nodeMCU/sensorweb-nodeMCU.sch (KiCad schematic (older format))
At the start: 19 parts, among them P1 PMS3003, Q1 2N2222, U1 LT1302CN8-5

Commit message: Fixing schematic and PCB
Parts:
- L1: footprint Inductors:INDUCTOR_V -> Inductors_NEOSID:Neosid_Inductor_Sd14
- Q1: footprint TO_SOT_Packages_THT:TO-18_3Pin -> TO_SOT_Packages_THT:TO-92_Inline_Narrow_Oval; symbol Q_NPN_BCE -> PN2222A
Connections:
- net +5V: now also C3.1, P1.8 (P8); no longer P1.1 (P1)
- net GND: now also C5.2, P1.7 (P7), Q1.1 (E); no longer C5.1, P1.2 (P2), Q1.3 (E)
- net at MCU1.18 (D10): now also P1.5 (P5); no longer P1.4 (P4)
- net at MCU1.19 (D9): now also P1.4 (P4); no longer P1.5 (P5)
- net at P1.6 (P6): now also Q1.3 (C), R2.2
- net at R1.1: now also Q1.2 (B); no longer Q1.1 (B)
- net at D1.2 (A), L1.1, U1.7 (SW): no longer C3.1
- net at B1.1 (P1), C1.1, C2.1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: now also C5.1; no longer C5.2
- now unconnected: P1.3 (P3)
Other:
- moved on the sheet: C3, D1
Changed lines of the file:
@@
 F 3 "" H 5900 2100 50  0000 C CNN
 	1    5900 2100
-	0    -1   -1   0
-$EndComp
-$Comp
-L Q_NPN_BCE Q1
+	0    1    -1   0
+$EndComp
+$Comp
+L PN2222A Q1
 U 1 1 586FE94A
-P 6950 2950
-F 0 "Q1" H 6900 2800 50  0000 R CNN
-F 1 "2N2222" H 7200 2750 50  0000 R CNN
-F 2 "TO_SOT_Packages_THT:TO-18_3Pin" H 7150 3050 50  0001 C CNN
-F 3 "" H 6950 2950 50  0000 C CNN
-	1    6950 2950
-	1    0    0    -1
+P 7000 2950
+F 0 "Q1" V 6850 2850 50  0000 R CNN
+F 1 "2N2222" V 7250 2900 50  0000 R CNN
+F 2 "TO_SOT_Packages_THT:TO-92_Inline_Narrow_Oval" H 7200 3050 50  0001 C CNN
+F 3 "" H 7000 2950 50  0000 C CNN
+	1    7000 2950
+	0    1    1    0
 $EndComp
 $Comp
@@
 F 0 "L1" V 3050 2100 50  0000 C CNN
 F 1 "22µH" V 3200 2100 50  0000 C CNN
-F 2 "Inductors:INDUCTOR_V" H 3100 2100 50  0001 C CNN
+F 2 "Inductors_NEOSID:Neosid_Inductor_Sd14" H 3100 2100 50  0001 C CNN
 F 3 "" H 3100 2100 50  0000 C CNN
 	1    3100 2100
@@
 L CP1 C3
 U 1 1 58753484
-P 2850 2550
-F 0 "C3" H 2875 2650 50  0000 L CNN
-F 1 "220µF" H 2875 2450 50  0000 L CNN
-F 2 "Capacitors_ThroughHole:C_Radial_D5_L6_P2.5" H 2850 2550 50  0001 C CNN
-F 3 "" H 2850 2550 50  0000 C CNN
-	1    2850 2550
+P 2600 2550
+F 0 "C3" H 2625 2650 50  0000 L CNN
+F 1 "220µF" H 2625 2450 50  0000 L CNN
+F 2 "Capacitors_ThroughHole:C_Radial_D5_L6_P2.5" H 2600 2550 50  0001 C CNN
+F 3 "" H 2600 2550 50  0000 C CNN
+	1    2600 2550
 	1    0    0    -1
 $EndComp
@@
 L D_Schottky D1
 U 1 1 58753565
-P 2500 2400
-F 0 "D1" H 2500 2500 50  0000 C CNN
-F 1 "1N5817" H 2500 2300 50  0000 C CNN
-F 2 "Diodes_ThroughHole:Diode_DO-41_SOD81_Horizontal_RM10" H 2500 2400 50  0001 C CNN
-F 3 "" H 2500 2400 50  0000 C CNN
-	1    2500 2400
+P 2900 2400
+F 0 "D1" H 2900 2500 50  0000 C CNN
+F 1 "1N5817" H 2900 2300 50  0000 C CNN
+F 2 "Diodes_ThroughHole:Diode_DO-41_SOD81_Horizontal_RM10" H 2900 2400 50  0001 C CNN
+F 3 "" H 2900 2400 50  0000 C CNN
+	1    2900 2400
 	1    0    0    -1
 $EndComp
@@
 L GND #PWR05
 U 1 1 587537D1
-P 2700 2700
-F 0 "#PWR05" H 2700 2450 50  0001 C CNN
-F 1 "GND" H 2700 2550 50  0000 C CNN
-F 2 "" H 2700 2700 50  0000 C CNN
-F 3 "" H 2700 2700 50  0000 C CNN
-	1    2700 2700
+P 2450 2700
+F 0 "#PWR05" H 2450 2450 50  0001 C CNN
+F 1 "GND" H 2450 2550 50  0000 C CNN
+F 2 "" H 2450 2700 50  0000 C CNN
+F 3 "" H 2450 2700 50  0000 C CNN
+	1    2450 2700
 	0    1    1    0
 $EndComp
@@
 L +5V #PWR06
 U 1 1 587537FF
-P 2300 2250
-F 0 "#PWR06" H 2300 2100 50  0001 C CNN
-F 1 "+5V" H 2300 2390 50  0000 C CNN
-F 2 "" H 2300 2250 50  0000 C CNN
-F 3 "" H 2300 2250 50  0000 C CNN
-	1    2300 2250
+P 2600 2300
+F 0 "#PWR06" H 2600 2150 50  0001 C CNN
+F 1 "+5V" H 2600 2440 50  0000 C CNN
+F 2 "" H 2600 2300 50  0000 C CNN
+F 3 "" H 2600 2300 50  0000 C CNN
+	1    2600 2300
 	1    0    0    -1
 $EndComp
@@
 F 3 "" H 1900 2650 50  0000 C CNN
 	1    1900 2650
-	-1   0    0    1
+	-1   0    0    -1
 $EndComp
 $Comp
@@
 $EndComp
 Wire Wire Line
-	7050 2650 7050 2750
-Wire Wire Line
-	7050 2700 6700 2700
+	6700 2700 7200 2700
 Wire Wire Line
 	6700 2700 6700 1900
@@
 Wire Wire Line
 	5750 2350 5750 2300
-Connection ~ 7050 2700
 Wire Wire Line
 	6350 2950 6400 2950
 Wire Wire Line
-	6700 2950 6750 2950
-Wire Wire Line
-	5000 4200 7050 4200
+	5000 4200 6800 4200
 Wire Wire Line
 	5350 4200 5350 3950
@@
 	5350 3850 5450 3850
 Wire Wire Line
-	5300 3950 5300 2400
+	5300 2400 5300 3950
 Wire Wire Line
 	5300 2400 5650 2400
@@
 	5550 2350 5550 2300
 Wire Wire Line
-	7050 4200 7050 3150
+	6800 4200 6800 3050
 Wire Wire Line
 	5850 2300 5850 2350
 Wire Wire Line
-	5850 2350 5800 2350
-Wire Wire Line
-	5800 2350 5800 1950
-Wire Wire Line
-	5800 1950 6600 1950
+	5850 2350 5900 2350
+Wire Wire Line
+	5900 2350 5900 1950
+Wire Wire Line
+	5900 1950 6600 1950
 Wire Wire Line
 	6600 1950 6600 3850
@@
 	3100 1800 3100 1450
 Connection ~ 3100 1450
-Wire Wire Line
-	2650 2400 3250 2400
-Connection ~ 2850 2400
-Connection ~ 3100 2400
-Wire Wire Line
-	2700 2700 2850 2700
-Wire Wire Line
-	2350 2400 2300 2400
-Wire Wire Line
-	2300 2400 2300 2250
 Wire Wire Line
 	3750 2950 3750 2950
@@
 	4950 2500 4900 2500
 Connection ~ 4900 2500
+Wire Wire Line
+	3050 2400 3250 2400
+Connection ~ 3100 2400
+Wire Wire Line
+	2600 2400 2750 2400
+Wire Wire Line
+	2600 2400 2600 2300
+Wire Wire Line
+	2450 2700 2600 2700
+Wire Wire Line
+	7000 2750 6750 2750
+Wire Wire Line
+	6750 2750 6750 2950
+Wire Wire Line
+	6750 2950 6700 2950
+Wire Wire Line
+	7200 2700 7200 3050
+Wire Wire Line
+	7050 2700 7050 2650
+Connection ~ 7050 2700
 $EndSCHEMATC
